File: Make Physical Things/IS250 Interface Board/5V-12V Signal Speedo.kicad_sch (KiCad schematic)
At the start: 3 parts

Commit message: Updated Components to have footprints
Added footprints to components that had the wrong ones or were completely missing
Parts:
- removed Q?: PN2222A, Package_TO_SOT_THT:TO-92_Inline, symbol Transistor_BJT:PN2222A
- removed R?: 4.7k, symbol Device:R
- added Q7: PN2222A, Package_TO_SOT_THT:TO-92_Inline, symbol Transistor_BJT:PN2222A
- added R12: 4.7k, Resistor_THT:R_Axial_DIN0207_L6.3mm_D2.5mm_P10.16mm_Horizontal, symbol Device:R
- gave numbers to parts that had none: 1
Connections:
- net GND: now also Q7.1 (E)
- net SPD IN: now also Q7.3 (C)
- net at U2.3 (Q0): now also R12.1
- new net: Q7.2 (B), R12.2
Changed lines of the file:
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@@
     (effects (font (size 1.27 1.27)) (justify left))
+  )
+  (symbol (lib_id "power:GND") (at 128.016 75.438 0) (unit 1)
+    (in_bom yes) (on_board yes) (fields_autoplaced)
+    (property "Reference" "#PWR0125" (id 0) (at 128.016 81.788 0)
+      (effects (font (size 1.27 1.27)) hide)
+    )
+    (property "Value" "GND" (id 1) (at 128.016 80.518 0))
+    (property "Footprint" "" (id 2) (at 128.016 75.438 0)
+      (effects (font (size 1.27 1.27)) hide)
+    )
+    (property "Datasheet" "" (id 3) (at 128.016 75.438 0)
+      (effects (font (size 1.27 1.27)) hide)
+    )
+    (pin "1")
   )
   (symbol (lib_id "Transistor_BJT:PN2222A") (at 125.476 67.818 0) (unit 1)
     (in_bom yes) (on_board yes) (fields_autoplaced)
-    (property "Reference" "Q?" (id 0) (at 130.556 66.5479 0)
+    (property "Reference" "Q7" (id 0) (at 130.556 66.5479 0)
       (effects (font (size 1.27 1.27)) (justify left))
     )
@@
     (pin "3")
   )
+  (symbol (lib_id "Device:R") (at 114.046 67.818 90) (unit 1)
+    (in_bom yes) (on_board yes) (fields_autoplaced)
+    (property "Reference" "R12" (id 0) (at 114.046 60.96 90))
+    (property "Value" "4.7k" (id 1) (at 114.046 63.5 90))
+    (property "Footprint" "Resistor_THT:R_Axial_DIN0207_L6.3mm_D2.5mm_P10.16mm_Horizontal" (id 2) (at 114.046 69.596 90)
+      (effects (font (size 1.27 1.27)) hide)
+    )
+    (property "Datasheet" "~" (id 3) (at 114.046 67.818 0)
+      (effects (font (size 1.27 1.27)) hide)
+    )
+    (pin "1")
+    (pin "2")
+  )
   (symbol (lib_id "power:GND") (at 71.12 35.56 0) (unit 1)
     (in_bom yes) (on_board yes) (fields_autoplaced)
-    (property "Reference" "#PWR?" (id 0) (at 71.12 41.91 0)
+    (property "Reference" "#PWR0124" (id 0) (at 71.12 41.91 0)
       (effects (font (size 1.27 1.27)) hide)
     )
@@
   (symbol (lib_id "power:+5V") (at 93.98 50.8 0) (unit 1)
     (in_bom yes) (on_board yes) (fields_autoplaced)
-    (property "Reference" "#PWR?" (id 0) (at 93.98 54.61 0)
+    (property "Reference" "#PWR0112" (id 0) (at 93.98 54.61 0)
       (effects (font (size 1.27 1.27)) hide)
     )
@@
     (pin "1")
   )
-  (symbol (lib_id "Device:R") (at 114.046 67.818 90) (unit 1)
-    (in_bom yes) (on_board yes) (fields_autoplaced)
-    (property "Reference" "R?" (id 0) (at 114.046 61.468 90))
-    (property "Value" "4.7k" (id 1) (at 114.046 64.008 90))
-    (property "Footprint" "" (id 2) (at 114.046 69.596 90)
-      (effects (font (size 1.27 1.27)) hide)
-    )
-    (property "Datasheet" "~" (id 3) (at 114.046 67.818 0)
-      (effects (font (size 1.27 1.27)) hide)
-    )
-    (pin "1")
-    (pin "2")
-  )
   (symbol (lib_id "4xxx:4017") (at 71.12 50.8 270) (unit 1)
     (in_bom yes) (on_board yes) (fields_autoplaced)
-    (property "Reference" "U?" (id 0) (at 90.17 44.2212 90))
+    (property "Reference" "U2" (id 0) (at 90.17 44.2212 90))
     (property "Value" "4017" (id 1) (at 90.17 46.7612 90))
     (property "Footprint" "" (id 2) (at 71.12 50.8 0)
@@
     (pin "9")
   )
-  (symbol (lib_id "power:GND") (at 128.016 75.438 0) (unit 1)
+  (symbol (lib_id "power:GND") (at 48.26 53.34 0) (unit 1)
     (in_bom yes) (on_board yes) (fields_autoplaced)
-    (property "Reference" "#PWR?" (id 0) (at 128.016 81.788 0)
+    (property "Reference" "#PWR0123" (id 0) (at 48.26 59.69 0)
       (effects (font (size 1.27 1.27)) hide)
     )
-    (property "Value" "GND" (id 1) (at 128.016 80.518 0))
-    (property "Footprint" "" (id 2) (at 128.016 75.438 0)
-      (effects (font (size 1.27 1.27)) hide)
-    )
-    (property "Datasheet" "" (id 3) (at 128.016 75.438 0)
-      (effects (font (size 1.27 1.27)) hide)
-    )
-    (pin "1")
-  )
-  (symbol (lib_id "power:GND") (at 48.26 53.34 0) (unit 1)
-    (in_bom yes) (on_board yes) (fields_autoplaced)
-    (property "Reference" "#PWR?" (id 0) (at 48.26 59.69 0)
-      (effects (font (size 1.27 1.27)) hide)
-    )

Commit message: Added components to PCB
Got all the components adding onto the PCB, and fixed pinname errors with the 2907
Parts:
- U2: footprint (none) -> Package_DIP:DIP-16_W7.62mm
Changed lines of the file:
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@@
     (property "Reference" "U2" (id 0) (at 90.17 44.2212 90))
     (property "Value" "4017" (id 1) (at 90.17 46.7612 90))
-    (property "Footprint" "" (id 2) (at 71.12 50.8 0)
+    (property "Footprint" "Package_DIP:DIP-16_W7.62mm" (id 2) (at 71.12 50.8 0)
       (effects (font (size 1.27 1.27)) hide)
     )
