File: Make Physical Things/IS250 Interface Board/Illumination_Circuit.kicad_sch (KiCad schematic)
At the start: 1 part

Commit message: Added components to PCB
Got all the components adding onto the PCB, and fixed pinname errors with the 2907
Parts:
- RV1: footprint (none) -> Potentiometer_THT:Potentiometer_Bourns_3386P_Vertical
Changed lines of the file:
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@@
       (effects (font (size 1.27 1.27)) (justify right))
     )
-    (property "Footprint" "" (id 2) (at 93.726 108.966 0)
+    (property "Footprint" "Potentiometer_THT:Potentiometer_Bourns_3386P_Vertical" (id 2) (at 93.726 108.966 0)
       (effects (font (size 1.27 1.27)) hide)
     )
