File: Make Physical Things/IS250 Interface Board/5V-12V Signal.kicad_sch (KiCad schematic)
At the start: 5 parts

Commit message: Updated Components to have footprints
Added footprints to components that had the wrong ones or were completely missing
Parts:
- Q11: renamed from Q?; footprint TO92-EBC -> Package_TO_SOT_THT:TO-92_Inline
- R16, R17, R18: renamed from R?; footprint (none) -> Resistor_THT:R_Axial_DIN0207_L6.3mm_D2.5mm_P10.16mm_Horizontal
- gave numbers to parts that had none: 1
Changed lines of the file:
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@@
   (symbol (lib_id "Device:R") (at 77.47 88.9 270) (mirror x)
     (in_bom yes) (on_board yes)
-    (property "Reference" "R?" (id 0) (at 77.47 83.312 90))
+    (property "Reference" "R18" (id 0) (at 77.47 83.312 90))
     (property "Value" "22k" (id 1) (at 77.47 85.852 90))
-    (property "Footprint" "" (id 2) (at 77.47 90.678 90)
+    (property "Footprint" "Resistor_THT:R_Axial_DIN0207_L6.3mm_D2.5mm_P10.16mm_Horizontal" (id 2) (at 77.47 90.678 90)
       (effects (font (size 1.27 1.27)) hide)
     )
@@
   (symbol (lib_id "Transistor_BJT:PN2222A") (at 68.58 96.52 0)
     (in_bom yes) (on_board yes) (fields_autoplaced)
-    (property "Reference" "Q?" (id 0) (at 73.66 95.2499 0)
+    (property "Reference" "Q10" (id 0) (at 73.66 95.2499 0)
       (effects (font (size 1.27 1.27)) (justify left))
     )
@@
   (symbol (lib_id "Device:R") (at 71.12 82.55 0) (mirror x)
     (in_bom yes) (on_board yes) (fields_autoplaced)
-    (property "Reference" "R?" (id 0) (at 68.58 81.2799 0)
+    (property "Reference" "R17" (id 0) (at 68.58 81.2799 0)
       (effects (font (size 1.27 1.27)) (justify right))
     )
@@
       (effects (font (size 1.27 1.27)) (justify right))
     )
-    (property "Footprint" "" (id 2) (at 69.342 82.55 90)
+    (property "Footprint" "Resistor_THT:R_Axial_DIN0207_L6.3mm_D2.5mm_P10.16mm_Horizontal" (id 2) (at 69.342 82.55 90)
       (effects (font (size 1.27 1.27)) hide)
     )
@@
   (symbol (lib_id "power:+12V") (at 83.82 88.9 0)
     (in_bom yes) (on_board yes) (fields_autoplaced)
-    (property "Reference" "#PWR?" (id 0) (at 83.82 92.71 0)
+    (property "Reference" "#PWR0132" (id 0) (at 83.82 92.71 0)
       (effects (font (size 1.27 1.27)) hide)
     )
@@
   (symbol (lib_id "PN2907A:PN2907A") (at 73.66 76.2 0)
     (in_bom yes) (on_board yes) (fields_autoplaced)
-    (property "Reference" "Q?" (id 0) (at 77.47 74.9045 0)
+    (property "Reference" "Q11" (id 0) (at 77.47 74.9045 0)
       (effects (font (size 1.27 1.27)) (justify left))
     )
@@
       (effects (font (size 1.27 1.27)) (justify left))
     )
-    (property "Footprint" "TO92-EBC" (id 2) (at 73.66 76.2 0)
+    (property "Footprint" "Package_TO_SOT_THT:TO-92_Inline" (id 2) (at 73.66 76.2 0)
       (effects (font (size 1.27 1.27)) (justify left bottom) hide)
     )
@@
   (symbol (lib_id "power:+12V") (at 76.2 68.58 0)
     (in_bom yes) (on_board yes) (fields_autoplaced)
-    (property "Reference" "#PWR0111" (id 0) (at 76.2 72.39 0)
+    (property "Reference" "#PWR0131" (id 0) (at 76.2 72.39 0)
       (effects (font (size 1.27 1.27)) hide)
     )
@@
   (symbol (lib_id "Device:R") (at 57.15 96.52 90)
     (in_bom yes) (on_board yes) (fields_autoplaced)
-    (property "Reference" "R?" (id 0) (at 57.15 90.17 90))
+    (property "Reference" "R16" (id 0) (at 57.15 90.17 90))
     (property "Value" "4.7k" (id 1) (at 57.15 92.71 90))
-    (property "Footprint" "" (id 2) (at 57.15 98.298 90)
+    (property "Footprint" "Resistor_THT:R_Axial_DIN0207_L6.3mm_D2.5mm_P10.16mm_Horizontal" (id 2) (at 57.15 98.298 90)
       (effects (font (size 1.27 1.27)) hide)
     )
@@
   (symbol (lib_id "power:GND") (at 71.12 104.14 0)
     (in_bom yes) (on_board yes) (fields_autoplaced)
-    (property "Reference" "#PWR?" (id 0) (at 71.12 110.49 0)
+    (property "Reference" "#PWR0130" (id 0) (at 71.12 110.49 0)
       (effects (font (size 1.27 1.27)) hide)
     )

Commit message: Added components to PCB
Got all the components adding onto the PCB, and fixed pinname errors with the 2907
Parts:
- renumbered Q10 to Q8, Q11 to Q9, R16 to R13, R17 to R14, R18 to R15
Connections:
- net +12V: now also Q9.1 (E); no longer Q9.E
- net 12V Out: now also Q9.3 (C); no longer Q9.C
- net at R14.2: now also Q9.2 (B); no longer Q9.B
Changed lines of the file:
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@@
   (symbol (lib_id "Device:R") (at 77.47 88.9 270) (mirror x)
     (in_bom yes) (on_board yes)
-    (property "Reference" "R18" (id 0) (at 77.47 83.312 90))
+    (property "Reference" "R15" (id 0) (at 77.47 83.312 90))
     (property "Value" "22k" (id 1) (at 77.47 85.852 90))
     (property "Footprint" "Resistor_THT:R_Axial_DIN0207_L6.3mm_D2.5mm_P10.16mm_Horizontal" (id 2) (at 77.47 90.678 90)
@@
   (symbol (lib_id "Transistor_BJT:PN2222A") (at 68.58 96.52 0)
     (in_bom yes) (on_board yes) (fields_autoplaced)
-    (property "Reference" "Q10" (id 0) (at 73.66 95.2499 0)
+    (property "Reference" "Q8" (id 0) (at 73.66 95.2499 0)
       (effects (font (size 1.27 1.27)) (justify left))
     )
@@
   (symbol (lib_id "Device:R") (at 71.12 82.55 0) (mirror x)
     (in_bom yes) (on_board yes) (fields_autoplaced)
-    (property "Reference" "R17" (id 0) (at 68.58 81.2799 0)
+    (property "Reference" "R14" (id 0) (at 68.58 81.2799 0)
       (effects (font (size 1.27 1.27)) (justify right))
     )
@@
   (symbol (lib_id "PN2907A:PN2907A") (at 73.66 76.2 0)
     (in_bom yes) (on_board yes) (fields_autoplaced)
-    (property "Reference" "Q11" (id 0) (at 77.47 74.9045 0)
+    (property "Reference" "Q9" (id 0) (at 77.47 74.9045 0)
       (effects (font (size 1.27 1.27)) (justify left))
     )
@@
       (effects (font (size 1.27 1.27)) (justify left bottom) hide)
     )
-    (pin "B")
-    (pin "C")
-    (pin "E")
+    (pin "2")
+    (pin "3")
+    (pin "1")
   )
   (symbol (lib_id "power:+12V") (at 76.2 68.58 0)
@@
   (symbol (lib_id "Device:R") (at 57.15 96.52 90)
     (in_bom yes) (on_board yes) (fields_autoplaced)
-    (property "Reference" "R16" (id 0) (at 57.15 90.17 90))
+    (property "Reference" "R13" (id 0) (at 57.15 90.17 90))
     (property "Value" "4.7k" (id 1) (at 57.15 92.71 90))
     (property "Footprint" "Resistor_THT:R_Axial_DIN0207_L6.3mm_D2.5mm_P10.16mm_Horizontal" (id 2) (at 57.15 98.298 90)

Commit message: Added XT60 and backup fuel resistor
Added an XT60 power connector, and an optional resistor if there isn't an AD8400 connected, so that the fuel gauge will show not empty
Parts:
- renumbered Q8 to Q10, Q9 to Q11, R13 to R16, R14 to R17, R15 to R18
Changed lines of the file:
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@@
   (symbol (lib_id "Device:R") (at 77.47 88.9 270) (mirror x)
     (in_bom yes) (on_board yes)
-    (property "Reference" "R15" (id 0) (at 77.47 83.312 90))
+    (property "Reference" "R18" (id 0) (at 77.47 83.312 90))
     (property "Value" "22k" (id 1) (at 77.47 85.852 90))
     (property "Footprint" "Resistor_THT:R_Axial_DIN0207_L6.3mm_D2.5mm_P10.16mm_Horizontal" (id 2) (at 77.47 90.678 90)
@@
   (symbol (lib_id "Transistor_BJT:PN2222A") (at 68.58 96.52 0)
     (in_bom yes) (on_board yes) (fields_autoplaced)
-    (property "Reference" "Q8" (id 0) (at 73.66 95.2499 0)
+    (property "Reference" "Q10" (id 0) (at 73.66 95.2499 0)
       (effects (font (size 1.27 1.27)) (justify left))
     )
@@
   (symbol (lib_id "Device:R") (at 71.12 82.55 0) (mirror x)
     (in_bom yes) (on_board yes) (fields_autoplaced)
-    (property "Reference" "R14" (id 0) (at 68.58 81.2799 0)
+    (property "Reference" "R17" (id 0) (at 68.58 81.2799 0)
       (effects (font (size 1.27 1.27)) (justify right))
     )
@@
   (symbol (lib_id "PN2907A:PN2907A") (at 73.66 76.2 0)
     (in_bom yes) (on_board yes) (fields_autoplaced)
-    (property "Reference" "Q9" (id 0) (at 77.47 74.9045 0)
+    (property "Reference" "Q11" (id 0) (at 77.47 74.9045 0)
       (effects (font (size 1.27 1.27)) (justify left))
     )
@@
       (effects (font (size 1.27 1.27)) (justify left bottom) hide)
     )
+    (pin "1")
     (pin "2")
     (pin "3")
-    (pin "1")
   )
   (symbol (lib_id "power:+12V") (at 76.2 68.58 0)
@@
   (symbol (lib_id "Device:R") (at 57.15 96.52 90)
     (in_bom yes) (on_board yes) (fields_autoplaced)
-    (property "Reference" "R13" (id 0) (at 57.15 90.17 90))
+    (property "Reference" "R16" (id 0) (at 57.15 90.17 90))
     (property "Value" "4.7k" (id 1) (at 57.15 92.71 90))
     (property "Footprint" "Resistor_THT:R_Axial_DIN0207_L6.3mm_D2.5mm_P10.16mm_Horizontal" (id 2) (at 57.15 98.298 90)

Commit message: More PCB Layout
PCB laid out further, and just requires routing and silkscreen.
Parts:
- renumbered Q10 to Q1, Q11 to Q2, R16 to R1, R18 to R11, R17 to R2
Changed lines of the file:
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@@
   (symbol (lib_id "Device:R") (at 77.47 88.9 270) (mirror x)
     (in_bom yes) (on_board yes)
-    (property "Reference" "R18" (id 0) (at 77.47 83.312 90))
+    (property "Reference" "R11" (id 0) (at 77.47 83.312 90))
     (property "Value" "22k" (id 1) (at 77.47 85.852 90))
     (property "Footprint" "Resistor_THT:R_Axial_DIN0207_L6.3mm_D2.5mm_P10.16mm_Horizontal" (id 2) (at 77.47 90.678 90)
@@
   (symbol (lib_id "Transistor_BJT:PN2222A") (at 68.58 96.52 0)
     (in_bom yes) (on_board yes) (fields_autoplaced)
-    (property "Reference" "Q10" (id 0) (at 73.66 95.2499 0)
+    (property "Reference" "Q1" (id 0) (at 73.66 95.2499 0)
       (effects (font (size 1.27 1.27)) (justify left))
     )
@@
   (symbol (lib_id "Device:R") (at 71.12 82.55 0) (mirror x)
     (in_bom yes) (on_board yes) (fields_autoplaced)
-    (property "Reference" "R17" (id 0) (at 68.58 81.2799 0)
+    (property "Reference" "R2" (id 0) (at 68.58 81.2799 0)
       (effects (font (size 1.27 1.27)) (justify right))
     )
@@
   (symbol (lib_id "PN2907A:PN2907A") (at 73.66 76.2 0)
     (in_bom yes) (on_board yes) (fields_autoplaced)
-    (property "Reference" "Q11" (id 0) (at 77.47 74.9045 0)
+    (property "Reference" "Q2" (id 0) (at 77.47 74.9045 0)
       (effects (font (size 1.27 1.27)) (justify left))
     )
@@
   (symbol (lib_id "Device:R") (at 57.15 96.52 90)
     (in_bom yes) (on_board yes) (fields_autoplaced)
-    (property "Reference" "R16" (id 0) (at 57.15 90.17 90))
+    (property "Reference" "R1" (id 0) (at 57.15 90.17 90))
     (property "Value" "4.7k" (id 1) (at 57.15 92.71 90))
     (property "Footprint" "Resistor_THT:R_Axial_DIN0207_L6.3mm_D2.5mm_P10.16mm_Horizontal" (id 2) (at 57.15 98.298 90)

Commit message: PCB Layout Finalised
Finalised the layout, routing and silkscreen still to be completed.
Parts:
- renumbered Q1 to Q10, Q2 to Q11, R1 to R16, R2 to R17, R11 to R18
Changed lines of the file:
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@@
   (symbol (lib_id "Device:R") (at 77.47 88.9 270) (mirror x)
     (in_bom yes) (on_board yes)
-    (property "Reference" "R11" (id 0) (at 77.47 83.312 90))
+    (property "Reference" "R18" (id 0) (at 77.47 83.312 90))
     (property "Value" "22k" (id 1) (at 77.47 85.852 90))
     (property "Footprint" "Resistor_THT:R_Axial_DIN0207_L6.3mm_D2.5mm_P10.16mm_Horizontal" (id 2) (at 77.47 90.678 90)
@@
   (symbol (lib_id "Transistor_BJT:PN2222A") (at 68.58 96.52 0)
     (in_bom yes) (on_board yes) (fields_autoplaced)
-    (property "Reference" "Q1" (id 0) (at 73.66 95.2499 0)
+    (property "Reference" "Q10" (id 0) (at 73.66 95.2499 0)
       (effects (font (size 1.27 1.27)) (justify left))
     )
@@
   (symbol (lib_id "Device:R") (at 71.12 82.55 0) (mirror x)
     (in_bom yes) (on_board yes) (fields_autoplaced)
-    (property "Reference" "R2" (id 0) (at 68.58 81.2799 0)
+    (property "Reference" "R17" (id 0) (at 68.58 81.2799 0)
       (effects (font (size 1.27 1.27)) (justify right))
     )
@@
   (symbol (lib_id "PN2907A:PN2907A") (at 73.66 76.2 0)
     (in_bom yes) (on_board yes) (fields_autoplaced)
-    (property "Reference" "Q2" (id 0) (at 77.47 74.9045 0)
+    (property "Reference" "Q11" (id 0) (at 77.47 74.9045 0)
       (effects (font (size 1.27 1.27)) (justify left))
     )
@@
   (symbol (lib_id "Device:R") (at 57.15 96.52 90)
     (in_bom yes) (on_board yes) (fields_autoplaced)
-    (property "Reference" "R1" (id 0) (at 57.15 90.17 90))
+    (property "Reference" "R16" (id 0) (at 57.15 90.17 90))
     (property "Value" "4.7k" (id 1) (at 57.15 92.71 90))
     (property "Footprint" "Resistor_THT:R_Axial_DIN0207_L6.3mm_D2.5mm_P10.16mm_Horizontal" (id 2) (at 57.15 98.298 90)
